Commit message: Added Wheels and Sensors

File: robot.urdf (robot description, URDF)
Before this commit: robot my_robot, 1 links, 0 joints
Links:
- added link castor_wheel; visual sphere radius=0.05
- added link left_wheel; visual cylinder length=0.05 radius=0.1
- added link right_wheel; visual cylinder length=0.05 radius=0.1
- added link sensor; visual cylinder length=0.05 radius=0.1
Joints:
- added joint base_castor_wheel_joint: type fixed, parent base_link, child castor_wheel, origin xyz=0.2 0 -0.05 rpy=0 0 0
- added joint base_left_wheel_joint: type continuous, parent base_link, child left_wheel, origin xyz=-0.15 0.225 0 rpy=0 0 0, axis 0 1 0
- added joint base_right_wheel_joint: type continuous, parent base_link, child right_wheel, origin xyz=-0.15 -0.225 0 rpy=0 0 0, axis 0 1 0
- added joint base_sensor_joint: type fixed, parent base_link, child sensor, origin xyz=0 0 0.225 rpy=0 0 0

Commit message: Added a base_footprint

File: robot.urdf (robot description, URDF)
Before this commit: robot my_robot, 5 links, 4 joints
Links:
- added link base_footprint
Joints:
- added joint base_joint: type fixed, parent base_link, child base_footprint, origin xyz=0 0 -0.1 rpy=0 0 0
